File: Design/Z31_HVAC_Disp_Rev1/Z31_HVAC_Disp_Rev1.kicad_pcb (KiCad board)
At the start: 0 parts

Commit message: large changes
Parts:
- added C1: 100n, Capacitor_SMD:C_0805_2012Metric_Pad1.18x1.45mm_HandSolder, B.Cu at (115.1, 96.0)
- added C2: 100n, Capacitor_SMD:C_0805_2012Metric_Pad1.18x1.45mm_HandSolder, B.Cu at (112.2, 74.7)
- added C3: 100n, Capacitor_SMD:C_0805_2012Metric_Pad1.18x1.45mm_HandSolder, F.Cu at (179.2, 81.7)
- added C4: 100n, Capacitor_SMD:C_0805_2012Metric_Pad1.18x1.45mm_HandSolder, B.Cu at (150.0, 97.9)
- added D1: LED, LED_THT:LED_Rectangular_W5.0mm_H2.0mm, F.Cu at (107.5, 68.4)
- added D10: LED, LED_THT:LED_Rectangular_W5.0mm_H2.0mm, F.Cu at (107.5, 84.6)
- added D11: LED, LED_THT:LED_Rectangular_W5.0mm_H2.0mm, F.Cu at (101.8, 87.3)
- added D12: LED, LED_THT:LED_Rectangular_W5.0mm_H2.0mm, F.Cu at (101.8, 90.0)
- added D13: LED, LED_THT:LED_Rectangular_W5.0mm_H2.0mm, F.Cu at (101.8, 92.7)
- added D14: LED, LED_THT:LED_Rectangular_W5.0mm_H2.0mm, F.Cu at (101.8, 95.4)
- added D15: LED, LED_THT:LED_Rectangular_W5.0mm_H2.0mm, F.Cu at (101.8, 98.1)
- added D16: LED, LED_THT:LED_Rectangular_W5.0mm_H2.0mm, F.Cu at (107.5, 98.1)
- added D2: LED, LED_THT:LED_Rectangular_W5.0mm_H2.0mm, F.Cu at (101.8, 68.4)
- added D3: LED, LED_THT:LED_Rectangular_W5.0mm_H2.0mm, F.Cu at (101.8, 71.1)
- added D4: LED, LED_THT:LED_Rectangular_W5.0mm_H2.0mm, F.Cu at (101.8, 73.8)
- added D5: LED, LED_THT:LED_Rectangular_W5.0mm_H2.0mm, F.Cu at (101.8, 76.5)
- added D6: LED, LED_THT:LED_Rectangular_W5.0mm_H2.0mm, F.Cu at (101.8, 79.2)
- added D7: LED, LED_THT:LED_Rectangular_W5.0mm_H2.0mm, F.Cu at (101.8, 81.9)
- added D8: LED, LED_THT:LED_Rectangular_W5.0mm_H2.0mm, F.Cu at (107.5, 81.9)
- added D9: LED, LED_THT:LED_Rectangular_W5.0mm_H2.0mm, F.Cu at (101.8, 84.6)
- added G***: LOGO, Personal:hvac overlay, F.Cu at (135.6, 82.3)
- added J1: Conn_01x18, Connector_PinSocket_2.54mm:PinSocket_1x18_P2.54mm_Vertical, B.Cu at (100.3, 65.4)
- added J2: Conn_01x10, Connector_PinSocket_2.54mm:PinSocket_1x10_P2.54mm_Vertical, B.Cu at (147.1, 65.4)
- added R1: 220, Resistor_SMD:R_0805_2012Metric, B.Cu at (113.5, 68.4)
- added R10: 220, Resistor_SMD:R_0805_2012Metric, B.Cu at (113.4, 84.6)
- added R11: 220, Resistor_SMD:R_0805_2012Metric, B.Cu at (107.7, 87.3)
- added R12: 220, Resistor_SMD:R_0805_2012Metric, B.Cu at (107.7, 90.0)
- added R13: 220, Resistor_SMD:R_0805_2012Metric, B.Cu at (107.7, 92.7)
- added R14: 220, Resistor_SMD:R_0805_2012Metric, B.Cu at (107.7, 95.4)
- added R15: 220, Resistor_SMD:R_0805_2012Metric, B.Cu at (111.3, 95.4)
- added R16: 220, Resistor_SMD:R_0805_2012Metric, B.Cu at (113.4, 98.1)
- added R17: 220, Resistor_SMD:R_0805_2012Metric, B.Cu at (142.4, 97.4)
- added R18: 220, Resistor_SMD:R_0805_2012Metric, B.Cu at (139.0, 96.1)
- added R19: 220, Resistor_SMD:R_0805_2012Metric, B.Cu at (142.4, 94.8)
- added R2: 220, Resistor_SMD:R_0805_2012Metric, B.Cu at (111.3, 71.1)
- added R20: 220, Resistor_SMD:R_0805_2012Metric, B.Cu at (139.0, 93.5)
- added R21: 220, Resistor_SMD:R_0805_2012Metric, B.Cu at (142.4, 92.2)
- added R22: 220, Resistor_SMD:R_0805_2012Metric, B.Cu at (139.0, 91.0)
- added R23: 220, Resistor_SMD:R_0805_2012Metric, B.Cu at (142.4, 89.7)
- added R24: 220, Resistor_SMD:R_0805_2012Metric, B.Cu at (139.0, 88.4)
- added R3: 220, Resistor_SMD:R_0805_2012Metric, B.Cu at (107.7, 71.1)
- added R4: 220, Resistor_SMD:R_0805_2012Metric, B.Cu at (107.7, 73.8)
- added R5: 220, Resistor_SMD:R_0805_2012Metric, B.Cu at (107.7, 76.5)
- added R6: 220, Resistor_SMD:R_0805_2012Metric, B.Cu at (107.7, 79.2)
- added R7: 220, Resistor_SMD:R_0805_2012Metric, B.Cu at (111.4, 79.2)
- added R8: 220, Resistor_SMD:R_0805_2012Metric, B.Cu at (113.4, 81.9)
- added R9: 220, Resistor_SMD:R_0805_2012Metric, B.Cu at (111.3, 87.3)
- added U1: 2.2__WVGA_SPI_14pin, LEDs:2.2_wvga_spi, F.Cu at (165.5, 82.9)
- added U2: 74HC595, Package_SO:SOIC-16_3.9x9.9mm_P1.27mm, B.Cu at (118.7, 73.3)
- added U3: 74HC595, Package_SO:SOIC-16_3.9x9.9mm_P1.27mm, B.Cu at (118.5, 91.2)
- added U4: 74HC595, Package_SO:SOIC-16_3.9x9.9mm_P1.27mm, B.Cu at (148.5, 91.6)
- added U5: CL3631AH, Personal:CL3631AH, F.Cu at (126.5, 91.5)
- added U6: CL3631AH, Personal:CL3631AH, F.Cu at (126.5, 73.0)
- added U7: ULN2003, Package_SO:SO-16_3.9x9.9mm_P1.27mm, B.Cu at (145.9, 74.4)
Routing:
- net GND: track 0.00 -> 98.5 mm, vias 0 -> 1
- net Net-(R17-Pad2): track 0.00 -> 50.7 mm, vias 0 -> 1
- net /LH_1: track 0.00 -> 48.4 mm, vias 0 -> 3
- net /LED_Dimming: track 0.00 -> 48.3 mm, vias 0 -> 2
- net Net-(R22-Pad2): track 0.00 -> 47.9 mm, vias 0 -> 1
- net Net-(R21-Pad2): track 0.00 -> 42.5 mm
- net Net-(R24-Pad2): track 0.00 -> 40.7 mm, vias 0 -> 1
- net Net-(U2-Pad9): track 0.00 -> 40.4 mm, vias 0 -> 2
- net Net-(J2-Pad4): track 0.00 -> 37.0 mm
- net Net-(R20-Pad2): track 0.00 -> 36.1 mm
- net Net-(R19-Pad2): track 0.00 -> 34.1 mm
- net Net-(J2-Pad5): track 0.00 -> 33.4 mm
- net Net-(R23-Pad2): track 0.00 -> 32.2 mm, vias 0 -> 1
- net Net-(R18-Pad2): track 0.00 -> 32.2 mm, vias 0 -> 1
- net Net-(J2-Pad6): track 0.00 -> 30.8 mm
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Other:
- board outline added: 100.5 x 45 mm
- copper layers 0 -> 2
