File: Design/Z31_HVAC_Disp_Rev1/Z31_HVAC_Disp_Rev1.kicad_sch (KiCad schematic)
At the start: 59 parts, among them J1 Conn_01x18, U1 74HC595, U2 74HC595, U3 74HC595, U4 CL3631AH, U5 CL3631AH, U6 ULN2003

Commit message: large changes
Connections:
- net GND: now also D1.1 (K), D10.1 (K), D11.1 (K), D12.1 (K), D13.1 (K), D14.1 (K), D15.1 (K), D16.1 (K), D2.1 (K), D3.1 (K), D4.1 (K), D5.1 (K), D6.1 (K), D7.1 (K), D8.1 (K), D9.1 (K)
